Commit message: feat: add saved pose controls and source-mounted development
Add session-scoped pose save and timed return with shared UI status, configurable duration, and independent inference resume. Make pose holds best-effort across command groups while retaining failed-stop interlocks.

Bind Cyclo-owned sources into runtime and worker containers, refresh robot description snapshots, and document rebuild requirements. Add runtime, RobotClient, UI, Docker, and Supervisor regression coverage.

Signed-off-by: kimtaehyeong99 <kth@robotis.com>

File: shared/shared/robot_configs/urdf/ffw_bg2_rev4_follower.urdf (robot description, URDF)
Before this commit: robot ffw_bg2_follower, 39 links, 38 joints
Links:
- added link end_effector_l_link; visual box size=0.01 0.01 0.01
- added link end_effector_r_link; visual box size=0.01 0.01 0.01
- link camera_l_link: geometry collision box size=0.023 0.042 0.042; visual mesh filename=file:///root/ros2_ws/install/realsense2_description/share/r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 scale=0.001 0.001 0.001
- link camera_r_link: geometry collision box size=0.023 0.042 0.042; visual mesh filename=file:///root/ros2_ws/install/realsense2_description/share/r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 scale=0.001 0.001 0.001
- link head_link1: mass 1.235180200e-01 -> 0.123518
Joints:
- added joint end_effector_l_joint: type fixed, parent arm_l_link7, child end_effector_l_link, origin xyz=0 0 -0.215 rpy=0 0 0
- added joint end_effector_r_joint: type fixed, parent arm_r_link7, child end_effector_r_link, origin xyz=0 0 -0.215 rpy=0 0 0
- joint gripper_l_joint: origin xyz=0 0 -0.078 rpy=0 3.14159265359 0 -> xyz=0 0 -0.078 rpy=0 3.14159265359 3.14159265359
- joint gripper_r_joint: origin xyz=0 0 -0.078 rpy=0 3.14159265359 0 -> xyz=0 0 -0.078 rpy=0 3.14159265359 3.14159265359
- joint head_joint1: limit lower=-0.2317 upper=0.6951 effort=1000 velocity=4.8 -> lower=-0.2317 upper=0.83 effort=1000 velocity=4.8; origin xyz=0.0494878 0 0.102123 rpy=0 0 0 -> xyz=0.049483 0 0.102130 rpy=0 0 0
- joint head_joint2: origin xyz=0.0365694 0 0.0563797 rpy=0 0 0 -> xyz=0.040 0 0.054 rpy=0 0 0

File: shared/shared/robot_configs/urdf/ffw_f1_follower.urdf (robot description, URDF)
Before this commit: robot ffw_f1_follower, 37 links, 36 joints
Links:
- removed link camera_l_base_link
- removed link camera_l_link
- removed link camera_r_base_link
- removed link camera_r_link
- added link camera_left_base_link, mass 3.6935029e-02; collision mesh filename=package://ffw_description/meshes/common/follower/wrist_d401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 scale=0.001 0.001 0.001; visual mesh filename=package://ffw_description/meshes/common/follower/wrist_d401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 scale=0.001 0.001 0.001
- added link camera_left_link
- added link camera_right_base_link, mass 3.6935029e-02; collision mesh filename=package://ffw_description/meshes/common/follower/wrist_d401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 scale=0.001 0.001 0.001; visual mesh filename=package://ffw_description/meshes/common/follower/wrist_d401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 scale=0.001 0.001 0.001
- added link camera_right_link
Joints:
- removed joint camera_l_joint
- removed joint camera_l_link_joint
- removed joint camera_r_joint
- removed joint camera_r_link_joint
- added joint camera_left_joint: type fixed, parent camera_left_base_link, child camera_left_link, origin xyz=0.0126724 -0.02235 0.009 rpy=0 0 0.3490656
- added joint camera_left_link_joint: type fixed, parent arm_l_link7, child camera_left_base_link, origin xyz=0.0275 0.0 -0.0847501 rpy=-1.57079632679 1.57079632679 0
- added joint camera_right_joint: type fixed, parent camera_right_base_link, child camera_right_link, origin xyz=0.0126724 -0.02235 0.009 rpy=0 0 0.3490656
- added joint camera_right_link_joint: type fixed, parent arm_r_link7, child camera_right_base_link, origin xyz=0.0275 0.0 -0.0847501 rpy=-1.57079632679 1.57079632679 0
- joint arm_l_joint7: limit lower=-1.8201 upper=1.5804 effort=1000 velocity=4.8 -> lower=-1.5804 upper=1.8201 effort=1000 velocity=4.8
- joint arm_r_joint7: limit lower=-1.5804 upper=1.8201 effort=1000 velocity=4.8 -> lower=-1.8201 upper=1.5804 effort=1000 velocity=4.8

File: shared/shared/robot_configs/urdf/ffw_f2_follower.urdf (robot description, URDF)
Before this commit: robot ffw_f2_follower, 46 links, 45 joints
Links:
- removed link camera_l_base_link
- removed link camera_l_link
- removed link camera_r_base_link
- removed link camera_r_link
- added link camera_left_base_link, mass 3.6935029e-02; collision mesh filename=package://ffw_description/meshes/common/follower/wrist_d401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 scale=0.001 0.001 0.001; visual mesh filename=package://ffw_description/meshes/common/follower/wrist_d401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 scale=0.001 0.001 0.001
- added link camera_left_link
- added link camera_right_base_link, mass 3.6935029e-02; collision mesh filename=package://ffw_description/meshes/common/follower/wrist_d401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 scale=0.001 0.001 0.001; visual mesh filename=package://ffw_description/meshes/common/follower/wrist_d401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 scale=0.001 0.001 0.001
- added link camera_right_link
- link arm_base_link: mass 7.0063905e+00 -> 7.0041009e+00
- link camera_head_link: geometry collision box size=0.026 0.124 0.029; visual mesh filename=file:///root/ros2_ws/install/realsense2_description/share/r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 scale=0.001 0.001 0.001
Joints:
- removed joint camera_l_joint
- removed joint camera_l_link_joint
- removed joint camera_r_joint
- removed joint camera_r_link_joint
- added joint camera_left_joint: type fixed, parent camera_left_base_link, child camera_left_link, origin xyz=0.0126724 -0.02235 0.009 rpy=0 0 0.3490656
- added joint camera_left_link_joint: type fixed, parent arm_l_link7, child camera_left_base_link, origin xyz=0.0275 0.0 -0.0847501 rpy=-1.57079632679 1.57079632679 0
- added joint camera_right_joint: type fixed, parent camera_right_base_link, child camera_right_link, origin xyz=0.0126724 -0.02235 0.009 rpy=0 0 0.3490656
- added joint camera_right_link_joint: type fixed, parent arm_r_link7, child camera_right_base_link, origin xyz=0.0275 0.0 -0.0847501 rpy=-1.57079632679 1.57079632679 0
- joint arm_l_joint7: limit lower=-1.8201 upper=1.5804 effort=1000 velocity=4.8 -> lower=-1.5804 upper=1.8201 effort=1000 velocity=4.8
- joint arm_r_joint7: limit lower=-1.5804 upper=1.8201 effort=1000 velocity=4.8 -> lower=-1.8201 upper=1.5804 effort=1000 velocity=4.8

File: shared/shared/robot_configs/urdf/ffw_sg2_follower.urdf (robot description, URDF)
Before this commit: robot ffw_sg2_follower, 50 links, 49 joints
Links:
- link head_link1: mass 1.235180200e-01 -> 0.123518
- link left_wheel_drive_link: geometry collision cylinder length=0.05 radius=0.0865; visual mesh filename=package://ffw_description/meshes/ffw_sg2_rev1_follower/left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 scale=0.001 0.001 0.001
- link lidar_l_link: mass None -> 0.1; geometry visual cylinder length=0.03 radius=0.03
- link lidar_r_link: mass None -> 0.1; geometry visual cylinder length=0.03 radius=0.03
- link lift_link: mass 1.790000000e+01 -> 17.9
- link rear_wheel_drive_link: geometry collision cylinder length=0.05 radius=0.0865; visual mesh filename=package://ffw_description/meshes/ffw_sg2_rev1_follower/rear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 scale=0.001 0.001 0.001
- link right_wheel_drive_link: geometry collision cylinder length=0.05 radius=0.0865; visual mesh filename=package://ffw_description/meshes/ffw_sg2_rev1_follower/righ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 scale=0.001 0.001 0.001
- link zedm_camera_center: geometry collision mesh filename=package://ffw_description/meshes/common/follower/zedm.stl scale=0.001 0.001 0.001; visual mesh filename=package://ffw_description/meshes/common/follower/zedm.stl scale=0.001 0.001 0.001
Joints:
- joint head_joint1: limit lower=-0.2317 upper=0.6951 effort=1000 velocity=4.8 -> lower=-0.2317 upper=0.83 effort=1000 velocity=4.8

File: shared/shared/robot_configs/urdf/ffw_sh5_follower.urdf (robot description, URDF)
Before this commit: robot ffw_sh5_follower, 90 links, 89 joints
Links:
- added link dummy_link1; visual box size=0.01 0.01 0.01
- added link dummy_link2; visual box size=0.01 0.01 0.01
- added link end_effector_l_link; visual box size=0.01 0.01 0.01
- added link end_effector_r_link; visual box size=0.01 0.01 0.01
- link base_link: mass 35.989 -> 3.598943900e+01
- link zedm_camera_center: geometry collision mesh filename=package://ffw_description/meshes/common/follower/zedm.stl scale=0.001 0.001 0.001; visual mesh filename=package://ffw_description/meshes/common/follower/zedm.stl scale=0.001 0.001 0.001
Joints:
- added joint end_effector_l_joint: type fixed, parent arm_l_link7, child end_effector_l_link, origin xyz=0 0 -0.215 rpy=0 0 0
- added joint end_effector_r_joint: type fixed, parent arm_r_link7, child end_effector_r_link, origin xyz=0 0 -0.215 rpy=0 0 0
- added joint gripper_l_joint1: type revolute, parent base_link, child dummy_link2, origin xyz=0.0 0.0 0.0 rpy=0 0 0, limit lower=-0.2317 upper=0.6951 effort=1000 velocity=4.8
- added joint gripper_r_joint1: type revolute, parent base_link, child dummy_link1, origin xyz=0.0 0.0 0.0 rpy=0 0 0, limit lower=-0.2317 upper=0.6951 effort=1000 velocity=4.8
- joint head_joint1: limit lower=-0.2317 upper=0.6951 effort=1000 velocity=4.8 -> lower=-0.2317 upper=0.83 effort=1000 velocity=4.8

File: shared/shared/robot_configs/urdf/omy_f3m.urdf (robot description, URDF)
Before this commit: robot omy_f3m, 17 links, 16 joints
Links:
- link camera_link: geometry collision box size=0.023 0.042 0.042; visual mesh filename=file:///root/ros2_ws/install/realsense2_description/share/r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 scale=0.001 0.001 0.001
